Commit message: update

File: body_v3/model3.urdf (robot description, URDF)
Before this commit: robot body_v3, 13 links, 12 joints
Links:
- link body:1: mass 0.3651787272540922 -> 1.497232781741777
- link link1_v2:1: mass 0.06405745692655854 -> 0.16654938800905217
- link link1_v2_(1):1: mass 0.06409335048954819 -> 0.1666427112728253
- link link1_v2_(2):1: mass 0.06409335048954819 -> 0.1666427112728253
- link link1_v2_(3):1: mass 0.06409335048954819 -> 0.1666427112728253
- link link2_v2:1: mass 0.009716027444754471 -> 0.025261671356361627
- link link2_v2_(1):1: mass 0.009716027444754475 -> 0.025261671356361634
- link link2_v2_(2):1: mass 0.009716027444754471 -> 0.025261671356361627
- link link2_v2_(3):1: mass 0.009750284046106812 -> 0.025350738519877708
- link link3_v2:1: mass 0.05868669884502759 -> 0.15258541699707173
- link link3_v2_(1):1: mass 0.05868669884502759 -> 0.15258541699707173
- link link3_v2_(2):1: mass 0.05868669884502759 -> 0.15258541699707173
- link link3_v2_(3):1: mass 0.05865244224367525 -> 0.15249634983355564
